File: Hardware/Schematic_PCB/ESP32_radio_rev1.0.brd (EAGLE design)
At the start: 160 x 56 mm, 35 parts, among them CON1 ENCODER1, CON2 ENCODER2, CON3 OLED Display, CON4 SD Card, CON5 Audio, CON6 JOY / SWITCHES

Commit message: Update
Parts:
- added C12: 10nF, rcl:C0603
- added C8: 100nF, rcl:C0603
- added SV1: KEYBOARD, con-lstb:MA04-1
- added SV2, USB2MODULE: (no value), con-lstb:MA03-1
- added SV3: SUB-C, con-lstb:MA06-1
- C14: value 220uF/6.3V -> 10uF/6.3V
- C16: value 220uF/6.3V -> 220uF/16V
- moved U$1 67.5 mm to (110.5, 50.8), turned to 0 degrees
- moved U$2 49.8 mm to (62.2, 22.9), turned to 0 degrees
- moved CON2 46.6 mm to (61.0, 76.2), turned to 0 degrees
- moved C7 45.7 mm to (33.0, 6.35), turned to 270 degrees
- moved C11 44.4 mm to (89.5, 47.6), turned to 270 degrees
- moved CON5 43.8 mm to (57.1, 48.3), turned to 90 degrees
- moved C10 41.0 mm to (85.7, 49.5), turned to 180 degrees
- moved R2 39.4 mm to (143.5, 49.5), turned to 270 degrees
- moved C13 39.1 mm to (57.1, 69.8)
- moved C16 29.0 mm to (66.0, 14.0)
- moved CON4 27.9 mm to (139.7, 15.2)
- moved CON1 24.2 mm to (78.7, 76.2), turned to 0 degrees
- moved H2 24.0 mm to (155.0, 75.0)
- moved CON3 23.0 mm to (138.4, 76.2), turned to 180 degrees
- moved C5 19.4 mm to (52.1, 3.81), turned to 270 degrees
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Connections:
- net BCK renamed N$15
- net LCK renamed N$10
- new net I2C: SV1.2, U$1.8
- new net I2C_ADC: SV1.1, U$1.9
- new net N$14: U$1.13, U$2.DIN
- new net N$18: SV2.1, U$1.15
- net +3V3: now also SV1.3, SV2.2; no longer C16.+
- net +5V: now also C12.2, C16.+, C8.2, SV3.6
- net DIN: no longer U$1.13, U$2.DIN
- net GND: now also C12.1, C8.1, SV1.4, SV2.3, SV3.1, U$2.SCK
Other:
- board size 160 x 56 mm -> 160 x 80 mm

Commit message: Schematic & PCB update
Parts:
- removed C16: 220uF/16V, rcl:150CLZ-1010
- removed CON1: ENCODER1, con-lsta:FE05-1
- removed CON2: ENCODER2, con-lsta:FE05-1
- removed CON3: OLED Display, con-lsta:FE07
- removed CON4: SD Card, con-lsta:FE06
- removed CON5: Audio, con-lstb:MA03-1
- removed CON6: JOY / SWITCHES, con-lsta:FE05-1
- removed H4: MOUNT-HOLE3.3, holes:3,3
- removed SV1: KEYBOARD, con-lstb:MA04-1
- removed SV2, USB2MODULE: (no value), con-lstb:MA03-1
- removed SV3: SUB-C, con-lstb:MA06-1
- removed U$2: I2S_PCM_51XX_SOUNDCARD, PCM5102A:I2S_PCM_5100_SOUNDCARD
- added *C8: 10nF, rcl:C0603
- added *R8, R10, R11, R14: 10k, rcl:R0603
- added 1: (no value), con-goldpins:MA10-1
- added 11, SV4: (no value), con-goldpins:MA12-1
- added AUDIO-OUT: AUDIO-OUT, JST XH Connectors v1-0:JST-XH-03-PACKAGE-LONG-PAD
- added C18, C19, C20, C21, C22: 100n, rcl:C0603
- added CARD: SD Card, JST XH Connectors v1-0:JST-XH-06-PACKAGE-LONG-PAD
- added D1: 5V, led:CHIP-LED0805
- added D2: 3.3V, led:CHIP-LED0805
- added EN1: ENCODER 1, JST XH Connectors v1-0:JST-XH-05-PACKAGE-LONG-PAD
- added EN2: ENCODER 2, JST XH Connectors v1-0:JST-XH-05-PACKAGE-LONG-PAD
- added H7, H8: MOUNT-HOLE3.3, holes:3,3
- added I2S: (no value), JST XH Connectors v1-0:JST-XH-06-PACKAGE-LONG-PAD
- added IR: IR, JST XH Connectors v1-0:JST-XH-03-PACKAGE-LONG-PAD
- added J1: (no value), jumper:SJ_2
- added J2, J3, J4, J5: (no value), jumper:SJ
- added JOY: JOY, JST XH Connectors v1-0:JST-XH-05-PACKAGE-LONG-PAD
- added KB: KYBOARD, JST XH Connectors v1-0:JST-XH-04-PACKAGE-LONG-PAD
- added L-OUT, R-OUT: TOBU3, con-hirschmann:TOBU3
- added M2: I2S_PCM_51XX_SOUNDCARD, PCM5102A:I2S_PCM_5100_SOUNDCARD
- added OLED: OLED, JST XH Connectors v1-0:JST-XH-07-PACKAGE-LONG-PAD
- added PW_SW: PWR_SWITCH, JST XH Connectors v1-0:JST-XH-02-PACKAGE-LONG-PAD
- added R12: 0, rcl:R0603
- added R13: 2k2, rcl:R0603
- added R16, R19, R20, R21: 10, rcl:R0603
- added R17, R18: 5.11k, rcl:R0603
- added R9: 100k, rcl:R0603
- added SD1: TF-HOLDER, sd-mmc:TF-PULL
- added SV7: (no value), con-lstb:MA10-1
- added U1: ESD Diode, SparkFun-DiscreteSemi:SOT-23-6
- added UBS2: PWR, JST XH Connectors v1-0:JST-XH-06-PACKAGE-LONG-PAD
- added USB: USB Data, JST XH Connectors v1-0:JST-XH-02-PACKAGE-LONG-PAD
- added USB-C: 2171790001, USB-C_2:2171790001_MOL
- C10, C11, C13, C9: value 33nF -> 10n
- C12: value 10nF -> 100n
- C14: device rcl:150CLZ-1010 -> rcl:C1210
- C15, C17: value 100nF -> 100n
- C8: value 100nF -> 10uF/6.3V; device rcl:C0603 -> rcl:C1210
- R7: value 4K7 -> 4k7
- R8: value 10k -> 2k2
- moved C12 137.8 mm to (132.0, 24.5)
- moved C8 135.1 mm to (132.0, 20.7), turned to 180 degrees
- moved C1 89.4 mm to (70.0, 5.50)
- moved C3 86.7 mm to (70.0, 9.50)
- moved C2 86.0 mm to (70.0, 7.50)
- moved C17 62.5 mm to (62.9, 61.0), turned to 270 degrees
- moved R6 57.2 mm to (62.9, 57.0), turned to 270 degrees
- moved R5 53.1 mm to (59.7, 52.6)
- moved R7 51.5 mm to (59.7, 57.8)
- moved R4 50.1 mm to (62.9, 53.5), turned to 90 degrees
- moved C9 46.1 mm to (62.7, 69.8), turned to 0 degrees
- moved R8 45.8 mm to (87.4, 15.0), turned to 90 degrees
- moved C11 44.0 mm to (51.5, 69.8), turned to 0 degrees
- moved C10 43.1 mm to (47.7, 69.8)
- moved C7 41.3 mm to (73.0, 16.5), turned to 180 degrees
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Connections:
- removed net CLK: R1.1, U$1.38
- removed net CS: CON3.7, U$1.42
- removed net DC: R3.1, U$1.40
- removed net DIN: R2.1, U$1.39
- removed net I2C: SV1.2, U$1.8
- removed net I2C_ADC: SV1.1, U$1.9
- removed net RESET: CON3.6, U$1.41
- new net 5V_USB: PW_SW.1, U1.5, UBS2.6, USB-C.A4/B9, USB-C.B4/A9
- new net ANALOGGND: AUDIO-OUT.2, L-OUT.2, L-OUT.2@1, L-OUT.2@2, M2.G2, R-OUT.2, R-OUT.2@1, R-OUT.2@2
- new net FMT: M2.4, R12.2
- new net FMT1: 11.4, U$1.46
- new net I2C-SCL-ADC: *C8.1, 11.5, KB.2, R11.1, R9.1, U$1.9
- new net I2C-SDA: 11.2, KB.1, R10.1, U$1.8
- new net N$12: R20.2, SD1.2
- new net N$16: 1.7, U$1.7
- new net N$17: SV7.6, U$1.2
- new net N$19: D2.C, R8.2
- new net N$20: SV7.8, U$1.44
- new net N$21: SV7.9, U$1.43
- new net N$22: SV4.3, U$1.19
- new net N$23: SV4.4, U$1.20
- new net N$24: SV4.9, U$1.0
- new net N$25: SV4.10, U$1.35
- new net N$26: SV4.11, U$1.36
- new net N$27: SV4.12, U$1.37
- new net N$28: 11.3, R12.1, U$1.3
- new net N$30: D1.C, R13.2
- new net N$31: CARD.1, J1.2
- new net N$32: R19.2, SD1.3
- new net N$33: R16.2, SD1.5
- new net N$34: U1.3, UBS2.5, USB-C.A6, USB-C.B6, USB.2
- new net N$35: U1.1, UBS2.4, USB-C.A7, USB-C.B7, USB.1
- new net N$36: I2S.3, J2.2
- new net N$37: R17.2, U1.4, UBS2.2, USB-C.B5
- new net N$38: R18.2, U1.6, UBS2.3, USB-C.A5
- new net N$39: I2S.6, J3.2
- new net N$4: OLED.5, R1.2
- new net N$40: I2S.5, J5.2
- new net N$41: I2S.4, J4.2
- new net OLED-CLK: R1.1, SV7.1, U$1.38
- new net OLED-CS: OLED.1, SV7.5, U$1.42
- new net OLED-DC: R3.1, SV7.3, U$1.40
- new net OLED-MOSI: R2.1, SV7.2, U$1.39
- new net OLED-RESET: OLED.2, SV7.4, U$1.41
- net +3V3: now also *R8.1, 1.1, 1.2, C12.2, C14.1, C18.2, C19.2, C20.1, C21.1, C8.1, D2.A, EN1.4, EN2.4, IR.2, J1.3, JOY.2, KB.3, R10.2, R11.2, R14.2, R9.2, SD1.4; no longer C14.+, CON1.4, CON2.4, CON4.1, CON6.2, R8.1, SV1.3, SV2.2
- net +5V: now also 11.11, C22.2, D1.A, I2S.1, J1.1, M2.VIN, OLED.7, PW_SW.2; no longer C12.2, C16.+, C8.2, CON3.2, SV3.6, U$2.VIN
- net CLK-A1: now also 1.6, EN1.1; no longer CON1.1
- net CLK-A2: now also 11.6, EN2.1; no longer CON2.1
- net CLK-SD: now also CARD.2, R16.1, SV4.8; no longer CON4.2
- net CS-SD: now also CARD.4, R20.1, SV4.6; no longer CON4.4
- net DT-B1: now also 1.5, EN1.2; no longer CON1.2
- net DT-B2: now also 11.7, EN2.2; no longer CON2.2
- net GND: now also *C8.2, 11.12, C14.2, C18.1, C19.1, C20.2, C21.2, C22.1, C8.2, CARD.6, EN1.5, EN2.5, I2S.2, IR.3, JOY.1, KB.4, M2.GND, M2.SCK, OLED.6, R13.1, R17.1, R18.1, R8.1, SD1.6, SD1.S1, SD1.S2, SD1.S3, SD1.S4, SV4.1, SV4.2, SV7.10, U1.2, UBS2.1, USB-C.A1/B12, USB-C.B1/A12; no longer C14.-, C16.-, C8.1, CON1.5, CON2.5, CON3.1, CON4.6, CON6.1, SV1.4, SV2.3, SV3.1, U$2.GND, U$2.SCK
- net MISO-SD: now also CARD.5, R21.1, SV4.5; no longer CON4.5
- net MOSI-SD: now also CARD.3, R19.1, SV4.7; no longer CON4.3
- net N$1: now also AUDIO-OUT.1, M2.R, R-OUT.1; no longer CON5.1, U$2.R
- net N$10: now also 11.10, J2.1, M2.LCK; no longer U$2.LCK
- net N$11: now also *R8.2, 1.3; no longer R8.2
- net N$13: now also 1.9, JOY.4; no longer CON6.4
- net N$14: now also 11.9, J4.1, M2.DIN; no longer U$2.DIN
- net N$15: now also 11.8, J5.1, M2.BCK; no longer U$2.BCK
- net N$18: now also 1.8, IR.1, R14.1; no longer SV2.1
- net N$2: now also M2.G1; no longer CON5.2, U$2.G2
- net N$3: now also AUDIO-OUT.3, L-OUT.1, M2.L; no longer CON5.3, U$2.L
- net N$5: now also OLED.4, R2.2; no longer CON3.3, R1.2
- net N$6: now also OLED.3; no longer CON3.5
- net N$7: now also R21.2, SD1.7; no longer CON3.4, R2.2
- net N$8: now also 1.10, JOY.3; no longer CON6.3
- net N$9: now also 11.1, J3.1, JOY.5; no longer CON6.5
- net SW1: now also 1.4, EN1.3; no longer CON1.3
- net SW2: now also EN2.3, SV7.7; no longer CON2.3
Routing:
- net GND: track 0.00 -> 600.6 mm, vias 0 -> 19
- net +3V3: track 0.00 -> 424.5 mm, vias 0 -> 12
- net +5V: track 0.00 -> 208.7 mm, vias 0 -> 4
- net I2C-SCL-ADC: track 0.00 -> 88.7 mm
- net I2C-SDA: track 0.00 -> 77.4 mm
- net DT-B2: track 0.00 -> 69.3 mm
- net N$18: track 0.00 -> 60.4 mm
- net CLK-A2: track 0.00 -> 58.2 mm
- net SW2: track 0.00 -> 52.2 mm
- net 5V_USB: track 0.00 -> 48.7 mm, vias 0 -> 3
- net DT-B1: track 0.00 -> 47.8 mm, vias 0 -> 2
- net N$9: track 0.00 -> 47.3 mm, vias 0 -> 1
- net SW1: track 0.00 -> 45.2 mm, vias 0 -> 2
- net CLK-A1: track 0.00 -> 43.8 mm
- net N$15: track 0.00 -> 43.2 mm, vias 0 -> 1
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- added copper zone on layer 16, net ANALOGGND
Other:
- board size 160 x 80 mm -> 175 x 80 mm
- board text added: "175mm extentsion for 3D printed housing"
- board text added: "3.3V/ 5V"
- board text added: "3V3"
- board text added: "5V"
- board text added: "A"
- board text added: "ADC"
- board text added: "B"
- board text added: "BCK"
- board text added: "CLK"
- board text added: "CS"
- board text added: "DATA"
- board text added: "DC"
- board text added: "ESP32 Web Radio"
- board text added: "EXTENSION 175mm"
- board text added: "GND"
- board text added: "IN"
- board text added: "L"
- board text added: "LCK"
- board text added: "MCLK"
- board text added: "MISO"
- board text added: "MOSI"
- board text added: "PCB Rev 1.0 FEB 2025, Robgold, OPEN SOURCE"
- board text added: "PCM5102A module"
- board text added: "R"
- board text added: "RST"
- board text added: "SDA"
- board text added: "SW"
- board text added: "VCC"
- board text added: "https://github.com/dzikakuna"
- board text added: "https://www.elektroda.pl/rtvforum/topic4041603.html"
