File: Hardware/Schematic_PCB/Release_rev1.0/ESP32_radio_rev1.0.brd (EAGLE design)
At the start: 175 x 80 mm, 78 parts, among them M2 I2S_PCM_51XX_SOUNDCARD, U1 ESD Diode

Commit message: Update
Parts:
- added *R1, *R2, *R3, *R4: 10k, rcl:R0603
- moved USB 1.27 mm to (98.5, 16.5), turned to 0 degrees
- moved L-OUT 0.72 mm to (26.3, 7.20)
- moved R-OUT 0.31 mm to (41.3, 7.20)
Connections:
- net N$34 renamed DP
- net N$35 renamed DN
- net +3V3: now also *R1.1, *R2.1, *R3.1, *R4.1
- net N$12: now also *R1.2
- net N$32: now also *R2.2
- net N$33: now also *R3.2
- net N$7: now also *R4.2
Routing:
- net +3V3: track 424.5 -> 449.4 mm, vias 12 -> 14
- net ANALOGGND: track 12.6 -> 5.96 mm
- net DP: track 42.8 -> 38.3 mm
- net DN: track 36.9 -> 41.2 mm
- net N$3: track 17.0 -> 19.7 mm
- net N$1: track 17.1 -> 19.7 mm
- net N$7: track 22.1 -> 24.4 mm
- net N$33: track 30.8 -> 32.8 mm
- net GND: track 600.6 -> 601.2 mm
- net N$32: track 31.3 -> 30.8 mm, vias 0 -> 2
- net N$12: track 29.3 -> 29.1 mm, vias 2 -> 4
Other:
- board text added: "3.3V/5V"
- board text added: "DN DP"
- board text removed: "3.3V/ 5V"
- board text removed: "L"
- board text removed: "R"
