File: Hardware/Schematic_PCB/Release_rev1.0/ESP32_radio_rev1.0.sch (EAGLE design)
At the start: 75 parts, among them M2 I2S_PCM_51XX_SOUNDCARD, U1 ESD Diode

Commit message: Update
Parts:
- added *R1, *R2, *R3, *R4: 10k, rcl:R-EU_R0603
Connections:
- net N$34 renamed DP
- net N$35 renamed DN
- net +3V3: now also *R1.1, *R2.1, *R3.1, *R4.1
- net N$12: now also *R1.2
- net N$32: now also *R2.2
- net N$33: now also *R3.2
- net N$7: now also *R4.2
Other:
- moved on the sheet: PW_SW-1, PW_SW-2, R17, R18, SD1, U1, UBS2-1, UBS2-2, UBS2-3, UBS2-4, UBS2-5, UBS2-6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
